Commit message: Initial commit

File: add_post_pro_robot/urdf/multisensor_holder.urdf.xacro (robot description, xacro)
@@ -48,9 +48,11 @@
 		<origin rpy="0.000000 0.000000 0.000000" xyz="0.000000 0.000000 0.000000"/>
 	</joint>
+	<!--Changes here!-->
 	<joint name="end_effector_magnet" type="fixed">
 		<parent link="J6"/>
 		<child link="EEF_sensor_holder"/>
-		<origin rpy="0.000000 0.000000 ${M_PI}" xyz="0.000000 0.000000 0.000000"/>
+		<origin rpy="0.000000 0.00000 ${225*M_PI/180}" xyz="0.000000 0.000000 0.000000"/>
 	</joint>
+	<!--Changes here!-->
     <joint name="end_effector_scanner_holder" type="fixed">
     	<parent link="EEF_sensor_holder"/>

File: add_post_pro_robot/urdf/scancontrol.xacro (robot description, xacro)
@@ -1,4 +1,5 @@
 <?xml version="1.0" encoding="UTF-8"?>
 <robot xmlns:xacro="http://www.ros.org/wiki/xacro">
+<xacro:property name="M_PI" value="3.1415926535897931" />
 <xacro:macro name="scancontrol2900-100" params="parent">
 <!-- DONE -->
@@ -24,13 +25,19 @@
 	</link>
     <link name="scancontrol2900-50_laser"/>
+    <link name = "true_laser"/>
     <joint name="end_effector_scanner" type="fixed">
     	<parent link="${parent}"/>
 		<child link="EEF_scancontrol"/>
-		<origin rpy="0.000000 0.000000 0.000000" xyz="0.000000 0.000000 0.000000"/>
+		<origin rpy="0.000000 0.0000 ${M_PI}" xyz="0.000000 0.000000 0.000000"/>
     </joint>
     <joint name="laser_joint" type="fixed">
         <parent link="EEF_scancontrol" />
         <child link="scancontrol2900-50_laser" />
-        <origin xyz="0 -0.0324522 -.0761366" rpy="0 ${M_PI/2} ${-M_PI/2}"/>
+        <origin xyz="0 -0.0324522 -.0761366" rpy="0 ${M_PI} 0"/>
+    </joint>
+    <joint name="imaginary_joint" type="fixed">
+        <parent link="scancontrol2900-50_laser" />
+        <child link="true_laser" />
+        <origin xyz="0 0 0" rpy="0 0 ${M_PI/2}"/>
     </joint>
         <!-- <origin xyz="0 -0.0324522 -.0761366" rpy="${M_PI} ${M_PI/2} ${M_PI/2}"/> -->
